File: docs/evidence/schematic-capture/ESP32_PWM_LED.kicad_sch (KiCad schematic)
At the start: 3 parts, among them U1 ESP32-WROOM-32

Commit message: Stage: 3. Schematic capture (KiCad) complete
Parts:
- R1: value 220 -> 100
- renumbered 12mA to LED1
Changed lines of the file:
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@@
 		(in_pos_files yes)
 		(dnp no)
-		(property "Reference" "12mA"
+		(property "Reference" "LED1"
 			(at 124.46 95.5675 0)
 			(show_name no)
@@
 			(project "ESP32_PWM_LED"
 				(path "/f26ee2fa-cdb6-4822-b85b-4ecde553fec1"
-					(reference "12mA")
+					(reference "LED1")
 					(unit 1)
 				)
@@
 			)
 		)
-		(property "Value" "220"
+		(property "Value" "100"
 			(at 139.7 81.2799 0)
 			(show_name no)
